File: eagle/sandwich/sandwich.sch (EAGLE design)
At the start: 118 parts, among them IC1 ATMEGA644-20PU, J1 AVR_SPI_PRG_6NS, Q1 20MHZ, Q2 MOSFET-NCHANNELFQP30N06L, Q3 MOSFET-NCHANNELFQP30N06L, T0 47k, T1 47k, T2 47k, T3 47k

Commit message: issue#5: added decoupling caps
Parts:
- added C27, C28, C29, C30, C31: 0.1uF, SparkFun-Capacitors:CAPPTH
Connections:
- net +5V: now also C27.2, C28.2, C29.2, C30.2, C31.2
- net GND: now also C27.1, C28.1, C29.1, C30.1, C31.1
Other:
- moved on the sheet: C12, C13, C14, C15, C16, C17, C18, C19, C20, C21, C22, C23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

Commit message: Changed all screw terminals to the smaller DG350
Parts:
- removed JP4, JP5: (no value), jumper:JP4Q
- removed X1, X13, X14, X15: (no value), con-wago-500:W237-4
- removed X10, X11, X12, X7, X8, X9: (no value), con-wago-500:W237-103
- removed X2, X3, X4, X5, X6: (no value), con-wago-500:W237-102
- added HEATER0, HEATER1, TEMP0, TEMP1, V+: DG3XX-02-3.5, degson:DG3XX-02-3.5
- added JP0: (no value), jumper:JP4Q
- added MOTOR0, MOTOR1, MOTOR2, MOTOR3: DG3XX-04-3.5, degson:DG3XX-04-3.5
- added SER0: (no value), SparkFun-Connectors:M06SIP
- added X_MAX, X_MIN, Y_MAX, Y_MIN, Z_MAX, Z_MIN: DG3XX-03-3.5, degson:DG3XX-03-3.5
- JP2: device SparkFun-Connectors:M06SIP -> jumper:JP4Q
Connections:
- net +5V: now also JP0.2, JP0.4, JP0.6, JP0.8, JP2.2, JP2.4, JP2.6, JP2.8, SER0.3, X_MAX-3.KL, X_MIN-3.KL, Y_MAX-3.KL, Y_MIN-3.KL, Z_MAX-3.KL, Z_MIN-3.KL; no longer JP2.3, JP4.2, JP4.4, JP4.6, JP4.8, JP5.2, JP5.4, JP5.6, JP5.8, X10-3.KL, X11-3.KL, X12-3.KL, X7-3.KL, X8-3.KL, X9-3.KL
- net GND: now also SER0.1, SER0.2, TEMP0-2.KL, TEMP1-2.KL, V+-1.KL, X_MAX-2.KL, X_MIN-2.KL, Y_MAX-2.KL, Y_MIN-2.KL, Z_MAX-2.KL, Z_MIN-2.KL; no longer JP2.1, JP2.2, X10-2.KL, X11-2.KL, X12-2.KL, X3-2.KL, X5-2.KL, X6-1.KL, X7-2.KL, X8-2.KL, X9-2.KL
- net MISO: now also Y_MAX-1.KL; no longer X9-1.KL
- net MOSI: now also X_MAX-1.KL; no longer X11-1.KL
- net N$15: now also HEATER0-2.KL; no longer X2-2.KL
- net N$18: now also JP0.1; no longer JP1.1
- net N$21: now also HEATER1-2.KL; no longer X4-2.KL
- net N$22: now also JP0.3; no longer JP1.3
- net N$23: now also JP0.5; no longer JP1.5
- net N$24: now also JP0.7; no longer JP1.7
- net N$25: now also SER0.6; no longer JP2.6
- net N$30: now also MOTOR1-4.KL; no longer X13-4.KL
- net N$31: now also MOTOR1-3.KL; no longer X13-3.KL
- net N$32: now also MOTOR1-2.KL; no longer X13-2.KL
- net N$33: now also MOTOR1-1.KL; no longer X13-1.KL
- net N$38: now also JP1.1; no longer JP3.1
- net N$39: now also JP1.3; no longer JP3.3
- net N$40: now also JP1.5; no longer JP3.5
- net N$41: now also JP1.7; no longer JP3.7
- net N$45: now also MOTOR2-4.KL; no longer X14-4.KL
- net N$46: now also MOTOR2-3.KL; no longer X14-3.KL
- net N$47: now also MOTOR2-2.KL; no longer X14-2.KL
- net N$48: now also MOTOR2-1.KL; no longer X14-1.KL
- net N$53: now also JP2.1; no longer JP4.1
- net N$54: now also JP2.3; no longer JP4.3
- net N$55: now also JP2.5; no longer JP4.5
- net N$56: now also JP2.7; no longer JP4.7
- net N$6: now also MOTOR0-4.KL; no longer X1-4.KL
- net N$60: now also MOTOR3-4.KL; no longer X15-4.KL
- net N$61: now also MOTOR3-3.KL; no longer X15-3.KL
- net N$62: now also MOTOR3-2.KL; no longer X15-2.KL
- net N$63: now also MOTOR3-1.KL; no longer X15-1.KL
- net N$68: now also JP3.1; no longer JP5.1
- net N$69: now also JP3.3; no longer JP5.3
- net N$7: now also MOTOR0-3.KL; no longer X1-3.KL
- net N$70: now also JP3.5; no longer JP5.5
- net N$71: now also JP3.7; no longer JP5.7
- net N$8: now also MOTOR0-2.KL; no longer X1-2.KL
- net N$9: now also MOTOR0-1.KL; no longer X1-1.KL
- net RESET: no longer C11.2
- net SCK: now also Y_MIN-1.KL; no longer X10-1.KL
- net SERIAL_RX: now also SER0.4; no longer JP2.4
- net SERIAL_TX: now also SER0.5; no longer JP2.5
- net TEMP0: now also TEMP0-1.KL; no longer X3-1.KL
- net TEMP1: now also TEMP1-1.KL; no longer X5-1.KL
- net V+: now also HEATER0-1.KL, HEATER1-1.KL, V+-2.KL; no longer X2-1.KL, X4-1.KL, X6-2.KL
- net X_MIN: now also X_MIN-1.KL; no longer X12-1.KL
- net Z_MAX: now also Z_MAX-1.KL; no longer X7-1.KL
- net Z_MIN: now also Z_MIN-1.KL; no longer X8-1.KL
Other:
- moved on the sheet: C11, JP1, JP3

Commit message: reorganized for 11x17 printability, added title and date text
Connections:
- net RESET: now also C11.2
Other:
- note added: "8 May 2013"
- note added: "Sandwich v0.00"
- moved on the sheet: C1, C10, C11, C12, C13, C14, C15, C16, C17, C18, C19, C2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

Commit message: AVR pin assignments are now the same as Gen7t. Motor enables are now combined.
Connections:
- removed net ENABLE0: IC1.PCINT20/TDO_PC4, U$1.ENABLE
- removed net ENABLE1: IC1.PCINT23/TOSC2_PC7, U$2.ENABLE
- removed net ENABLE2: IC1.PCINT5/ADC5_PA5, U$3.ENABLE
- removed net ENABLE3: IC1.PCINT2/ADC2_PA2, U$4.ENABLE
- removed net X_MIN: IC1.PCINT10/INT2/AIN0_PB2, X_MIN-1.KL
- new net AUX8: IC1.PCINT20/TDO_PC4
- new net AUX9: IC1.PCINT21/TDI_PC5
- new net ENABLE: IC1.PCINT7/ADC7_PA7, U$1.ENABLE, U$2.ENABLE, U$3.ENABLE, U$4.ENABLE
- new net TEMP2: IC1.PCINT0/ADC0_PA0
- new net Y_MAX: IC1.PCINT10/INT2/AIN0_PB2, Y_MAX-1.KL
- net DIR1: now also IC1.PCINT22/TOSC1_PC6; no longer IC1.PCINT21/TDI_PC5
- net DIR2: now also IC1.PCINT6/ADC6_PA6; no longer IC1.PCINT7/ADC7_PA7
- net MISO: now also X_MAX-1.KL; no longer Y_MAX-1.KL
- net MOSI: now also Y_MIN-1.KL; no longer X_MAX-1.KL
- net SCK: now also X_MIN-1.KL; no longer Y_MIN-1.KL
- net STEP1: now also IC1.PCINT23/TOSC2_PC7; no longer IC1.PCINT22/TOSC1_PC6
- net STEP2: now also IC1.PCINT5/ADC5_PA5; no longer IC1.PCINT6/ADC6_PA6
- net TEMP0: now also IC1.PCINT2/ADC2_PA2; no longer IC1.PCINT0/ADC0_PA0

Commit message: Changed all connectors except V+ and heaters to pin headers, removed axis max inputs
Parts:
- removed X_MAX, Y_MAX, Z_MAX: DG3XX-03-3.5, degson:DG3XX-03-3.5
- MOTOR0, MOTOR1, MOTOR2, MOTOR3: value DG3XX-04-3.5 -> (none); device degson:DG3XX-04-3.5 -> SparkFun-Connectors:M04LONGPADS
- TEMP0, TEMP1: value DG3XX-02-3.5 -> (none); device degson:DG3XX-02-3.5 -> SparkFun-Connectors:M02PTH3
- X_MIN, Y_MIN, Z_MIN: value DG3XX-03-3.5 -> (none); device degson:DG3XX-03-3.5 -> SparkFun-Connectors:M03LONGPADS
Connections:
- net +5V: now also X_MIN.1, Y_MIN.1, Z_MIN.1; no longer X_MAX-3.KL, X_MIN-3.KL, Y_MAX-3.KL, Y_MIN-3.KL, Z_MAX-3.KL, Z_MIN-3.KL
- net GND: now also TEMP0.1, TEMP1.1, X_MIN.2, Y_MIN.2, Z_MIN.2; no longer TEMP0-2.KL, TEMP1-2.KL, X_MAX-2.KL, X_MIN-2.KL, Y_MAX-2.KL, Y_MIN-2.KL, Z_MAX-2.KL, Z_MIN-2.KL
- net MISO: no longer X_MAX-1.KL
- net MOSI: now also Y_MIN.3; no longer Y_MIN-1.KL
- net N$30: now also MOTOR1.4; no longer MOTOR1-4.KL
- net N$31: now also MOTOR1.3; no longer MOTOR1-3.KL
- net N$32: now also MOTOR1.2; no longer MOTOR1-2.KL
- net N$33: now also MOTOR1.1; no longer MOTOR1-1.KL
- net N$45: now also MOTOR2.4; no longer MOTOR2-4.KL
- net N$46: now also MOTOR2.3; no longer MOTOR2-3.KL
- net N$47: now also MOTOR2.2; no longer MOTOR2-2.KL
- net N$48: now also MOTOR2.1; no longer MOTOR2-1.KL
- net N$6: now also MOTOR0.4; no longer MOTOR0-4.KL
- net N$60: now also MOTOR3.4; no longer MOTOR3-4.KL
- net N$61: now also MOTOR3.3; no longer MOTOR3-3.KL
- net N$62: now also MOTOR3.2; no longer MOTOR3-2.KL
- net N$63: now also MOTOR3.1; no longer MOTOR3-1.KL
- net N$7: now also MOTOR0.3; no longer MOTOR0-3.KL
- net N$8: now also MOTOR0.2; no longer MOTOR0-2.KL
- net N$9: now also MOTOR0.1; no longer MOTOR0-1.KL
- net SCK: now also X_MIN.3; no longer X_MIN-1.KL
- net TEMP0: now also TEMP0.2; no longer TEMP0-1.KL
- net TEMP1: now also TEMP1.2; no longer TEMP1-1.KL
- net Y_MAX: no longer Y_MAX-1.KL
- net Z_MAX: no longer Z_MAX-1.KL
- net Z_MIN: now also Z_MIN.3; no longer Z_MIN-1.KL

Commit message: Changed motor connectors back to screw terminals, added a fan output and routed the board layout.
Parts:
- added D3: (no value), SparkFun-DiscreteSemi:DIODEPTH
- added FAN: (no value), SparkFun-Connectors:M02PTH3
- added R56: (no value), resistor:R-US_0204/2V
- added T4: 2N2222, transistor:2N2222
- MOTOR0, MOTOR1, MOTOR2, MOTOR3: value (none) -> DG3XX-04-3.5; device SparkFun-Connectors:M04LONGPADS -> degson:DG3XX-04-3.5
Connections:
- removed net AUX7: IC1.PCINT17/SDA_PC1
- new net FAN: IC1.PCINT17/SDA_PC1, R56.1
- new net N$26: D3.A, FAN.2, T4.C
- new net N$73: R56.2, T4.B
- net +5V: now also X_MIN.3, Y_MIN.3, Z_MIN.3; no longer X_MIN.1, Y_MIN.1, Z_MIN.1
- net GND: now also T4.E, TEMP0.2, TEMP1.2; no longer TEMP0.1, TEMP1.1
- net MOSI: now also Y_MIN.1; no longer Y_MIN.3
- net N$30: now also MOTOR1-1.KL, U$2.OUT1A; no longer MOTOR1.4, U$2.OUT2B
- net N$31: now also MOTOR1-2.KL, U$2.OUT2A; no longer MOTOR1.3, U$2.OUT1B
- net N$32: now also MOTOR1-3.KL, U$2.OUT1B; no longer MOTOR1.2, U$2.OUT2A
- net N$33: now also MOTOR1-4.KL, U$2.OUT2B; no longer MOTOR1.1, U$2.OUT1A
- net N$45: now also MOTOR2-1.KL, U$3.OUT1A; no longer MOTOR2.4, U$3.OUT2B
- net N$46: now also MOTOR2-2.KL, U$3.OUT2A; no longer MOTOR2.3, U$3.OUT1B
- net N$47: now also MOTOR2-3.KL, U$3.OUT1B; no longer MOTOR2.2, U$3.OUT2A
- net N$48: now also MOTOR2-4.KL, U$3.OUT2B; no longer MOTOR2.1, U$3.OUT1A
- net N$6: now also MOTOR0-4.KL; no longer MOTOR0.4
- net N$60: now also MOTOR3-1.KL, U$4.OUT1A; no longer MOTOR3.4, U$4.OUT2B
- net N$61: now also MOTOR3-2.KL, U$4.OUT2A; no longer MOTOR3.3, U$4.OUT1B
- net N$62: now also MOTOR3-3.KL, U$4.OUT1B; no longer MOTOR3.2, U$4.OUT2A
- net N$63: now also MOTOR3-4.KL, U$4.OUT2B; no longer MOTOR3.1, U$4.OUT1A
- net N$7: now also MOTOR0-3.KL; no longer MOTOR0.3
- net N$8: now also MOTOR0-2.KL; no longer MOTOR0.2
- net N$9: now also MOTOR0-1.KL; no longer MOTOR0.1
- net SCK: now also X_MIN.1; no longer X_MIN.3
- net TEMP0: now also TEMP0.1; no longer TEMP0.2
- net TEMP1: now also TEMP1.1; no longer TEMP1.2
- net V+: now also D3.C, FAN.1
- net Z_MIN: now also Z_MIN.1; no longer Z_MIN.3
Other:
- note added: "14 May 2013"
- note added: "Fan output"
- note removed: "8 May 2013"
- moved on the sheet: TEMP0, TEMP1, X_MIN, Y_MIN, Z_MIN

Commit message: Changed trim pots to 4.7k
Parts:
- T0, T1, T2, T3: value 47k -> 4.7k
Other:
- note added: "15 May 2013"
- note removed: "14 May 2013"
Changed lines of the file:
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@@
 </layers>
 <schematic xreflabel="%F%N/%S.%C%R" xrefpart="/%S.%C%R">
+<description>Sandwich v0.00
+low cost CNC/3D printer controller</description>
 <attributes>
 </attributes>
@@
 <part name="R11" library="resistor" deviceset="R-US_" device="0204/2V" value="4.7k"/>
 <part name="SUPPLY21" library="supply2" deviceset="+5V" device=""/>
-<part name="T0" library="SparkFun-Electromechanical" deviceset="POT" device="TRIM" value="47k"/>
+<part name="T0" library="SparkFun-Electromechanical" deviceset="POT" device="TRIM" value="4.7k"/>
 <part name="R12" library="resistor" deviceset="R-US_" device="0204/2V" value="1k"/>
 <part name="R13" library="resistor" deviceset="R-US_" device="0204/2V" value="1k"/>
@@
 <part name="R29" library="resistor" deviceset="R-US_" device="0204/2V" value="4.7k"/>
 <part name="SUPPLY66" library="supply2" deviceset="+5V" device=""/>
-<part name="T1" library="SparkFun-Electromechanical" deviceset="POT" device="TRIM" value="47k"/>
+<part name="T1" library="SparkFun-Electromechanical" deviceset="POT" device="TRIM" value="4.7k"/>
 <part name="R30" library="resistor" deviceset="R-US_" device="0204/2V" value="1k"/>
 <part name="R31" library="resistor" deviceset="R-US_" device="0204/2V" value="1k"/>
@@
 <part name="R41" library="resistor" deviceset="R-US_" device="0204/2V" value="4.7k"/>
 <part name="SUPPLY83" library="supply2" deviceset="+5V" device=""/>
-<part name="T2" library="SparkFun-Electromechanical" deviceset="POT" device="TRIM" value="47k"/>
+<part name="T2" library="SparkFun-Electromechanical" deviceset="POT" device="TRIM" value="4.7k"/>
 <part name="R42" library="resistor" deviceset="R-US_" device="0204/2V" value="1k"/>
 <part name="R43" library="resistor" deviceset="R-US_" device="0204/2V" value="1k"/>
@@
 <part name="R53" library="resistor" deviceset="R-US_" device="0204/2V" value="4.7k"/>
 <part name="SUPPLY100" library="supply2" deviceset="+5V" device=""/>
-<part name="T3" library="SparkFun-Electromechanical" deviceset="POT" device="TRIM" value="47k"/>
+<part name="T3" library="SparkFun-Electromechanical" deviceset="POT" device="TRIM" value="4.7k"/>
 <part name="R54" library="resistor" deviceset="R-US_" device="0204/2V" value="1k"/>
 <part name="R55" library="resistor" deviceset="R-US_" device="0204/2V" value="1k"/>
@@
 <wire x1="10.16" y1="7.62" x2="10.16" y2="78.74" width="0.1524" layer="97" style="longdash"/>
 <text x="193.04" y="251.46" size="6.4516" layer="97">Sandwich v0.00</text>
-<text x="193.04" y="243.84" size="3.81" layer="97">14 May 2013</text>
+<text x="193.04" y="243.84" size="3.81" layer="97">15 May 2013</text>
 <text x="144.78" y="139.7" size="1.778" layer="97">Fan output</text>
 <wire x1="116.84" y1="147.32" x2="182.88" y2="147.32" width="0.1524" layer="97" style="longdash"/>
