File: eagle/sandwich/sandwich.sch (EAGLE design)
At the start: 124 parts, among them IC1 ATMEGA644-20PU, J1 AVR_SPI_PRG_6NS, Q1 20MHZ, Q2 MOSFET-NCHANNELFQP30N06L, Q3 MOSFET-NCHANNELFQP30N06L, T0 4.7k, T1 4.7k, T2 4.7k, T3 4.7k, T4 2N2222

Commit message: Updated TB6600 package, moved R56, changed 100uF caps to 16v, disabled GND and V+ thermals. Still needs TB6600HG layout adjustment and new routing
Parts:
- C12, C13, C17, C18, C22, C23, C3, C4: device SparkFun-Passives:CAP_POLPTH1 -> SparkFun-Passives:CAP_POLPTH2
- D3: value (none) -> 1N4004
- R56: value (none) -> 1k7
- U$1, U$2, U$3, U$4: value TB6600HQ -> TB6600HG; device tb6600hq:TB6600HQ -> tb6600hq:TB6600HG
Other:
- note added: "Sandwich v0.01"
- note removed: "Sandwich v0.00"
- moved on the sheet: C9

Commit message: Moved FAN to a PWM output
Parts:
- Q2, Q3: value MOSFET-NCHANNELFQP30N06L -> IRFZ44N
Connections:
- net AUX4: now also IC1.PCINT17/SDA_PC1; no longer IC1.PCINT30/OC2B/ICP_PD6
- net FAN: now also IC1.PCINT30/OC2B/ICP_PD6; no longer IC1.PCINT17/SDA_PC1
Other:
- note added: "29 June 2013"
- note added: "Sandwich v0.02"
- note removed: "15 May 2013"
- note removed: "Sandwich v0.01"
